File: kicad/firewaterburn_devkit.kicad_pcb (KiCad board)
At the start: 2 copper layers, 20 parts, among them P201 USB_C_Plug_USB2.0, Q201 SS8050-G, Q202 SS8050-G, SW201 SW_MEC_5G, SW202 SW_MEC_5G, U201 CP2102N-A01-GQFN28, U202 ESP32-WROOM-32

Commit message: wip
Parts:
- removed C201, C202, C204, C205, C207: 100n, Capacitor_SMD:C_0603_1608Metric_Pad1.08x0.95mm_HandSolder
- removed C203: 4.7µ, Capacitor_SMD:C_0603_1608Metric_Pad1.08x0.95mm_HandSolder
- removed C206: 22µ, Capacitor_SMD:C_0603_1608Metric_Pad1.08x0.95mm_HandSolder
- removed P201: USB_C_Plug_USB2.0, Connector_USB:USB_C_Receptacle_Amphenol_12401610E4-2A
- removed Q201, Q202: SS8050-G, Package_TO_SOT_SMD:SOT-23
- removed R201, R202, R206: 10k, Resistor_SMD:R_0603_1608Metric_Pad0.98x0.95mm_HandSolder
- removed R203: 22k1, Resistor_SMD:R_0603_1608Metric_Pad0.98x0.95mm_HandSolder
- removed R204: 47k5, Resistor_SMD:R_0603_1608Metric_Pad0.98x0.95mm_HandSolder
- removed R205: 2k, Resistor_SMD:R_0603_1608Metric_Pad0.98x0.95mm_HandSolder
- removed SW201, SW202: SW_MEC_5G, firewaterburn:PTS820J25MSMTRLFS
- removed U201: CP2102N-A01-GQFN28, Package_DFN_QFN:QFN-28-1EP_5x5mm_P0.5mm_EP3.35x3.35mm
- removed U202: ESP32-WROOM-32, RF_Module:ESP32-WROOM-32
- added D1: LED, LED_SMD:LED_0805_2012Metric_Pad1.15x1.40mm_HandSolder, F.Cu at (143.0, 84.2)
- added D2: LED, LED_SMD:LED_0805_2012Metric_Pad1.15x1.40mm_HandSolder, F.Cu at (167.0, 84.2)
- added J1: AudioJack2_SwitchT, z_connector:MJ-2523, F.Cu at (160.0, 94.0)
- added J2: AudioJack2_SwitchT, z_connector:MJ-2523, F.Cu at (150.0, 94.0)
- added R1: 130, Resistor_SMD:R_0805_2012Metric_Pad1.20x1.40mm_HandSolder, F.Cu at (153.5, 88.0)
- added R2: 130, Resistor_SMD:R_0805_2012Metric_Pad1.20x1.40mm_HandSolder, F.Cu at (156.5, 88.0)
- added R3: 2k49, Resistor_SMD:R_0805_2012Metric_Pad1.20x1.40mm_HandSolder, F.Cu at (155.2, 98.7)
- added R4: 3k24, Resistor_SMD:R_0805_2012Metric_Pad1.20x1.40mm_HandSolder, F.Cu at (150.0, 99.0)
- added R5: 2k49, Resistor_SMD:R_0805_2012Metric_Pad1.20x1.40mm_HandSolder, F.Cu at (150.0, 97.0)
- added R6: 4k02, Resistor_SMD:R_0805_2012Metric_Pad1.20x1.40mm_HandSolder, F.Cu at (161.5, 104.0)
- added R7: 2k49, Resistor_SMD:R_0805_2012Metric_Pad1.20x1.40mm_HandSolder, F.Cu at (163.5, 99.0)
- added R8: 2k26, Resistor_SMD:R_0805_2012Metric_Pad1.20x1.40mm_HandSolder, F.Cu at (161.5, 99.0)
- added U1: ESP-WROOM-32, z_ic:esp-wroom-32-devkit, F.Cu at (155.0, 107.0)
- added U2: LT6202, Package_TO_SOT_SMD:TSOT-23-5, F.Cu at (158.3, 99.0)
Routing:
- net GND: track 0.00 -> 84.7 mm, vias 0 -> 6
- net +3V3: track 0.00 -> 50.6 mm, vias 0 -> 4
- net Net-(R1-Pad2): track 0.00 -> 31.5 mm, vias 0 -> 1
- net /T_lin: track 0.00 -> 20.9 mm
- net Net-(J1-PadS): track 0.00 -> 19.9 mm, vias 0 -> 2
- net Net-(R2-Pad2): track 0.00 -> 13.7 mm, vias 0 -> 1
- net /T_op: track 0.00 -> 13.4 mm, vias 0 -> 1
- net Net-(D2-Pad2): track 0.00 -> 11.2 mm
- net Net-(D1-Pad2): track 0.00 -> 11.2 mm
- net Net-(R6-Pad1): track 0.00 -> 10.2 mm
- added copper zone on B.Cu, net GND
- added copper zone on F.Cu, net GND
Other:
- board outline added: 28 x 51 mm
