File: kicad/mcu_n_tft.kicad_sch (KiCad schematic)
At the start: 14 parts, among them J301 Conn_ARM_SWD_TagConnect_TC2030, J303 Conn_02x10_Odd_Even, U301 BL654, Y301 Crystal

Commit message: new board
Parts:
- R402, R404: Digikey RNCP0603FTD1K00 -> RNCP0603FTD1K00CT-ND
Changed lines of the file:
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@@
+      (effects (font (size 1.27 1.27)) hide)
+    )
+    (property "Digikey" "" (at 29.21 43.18 0)
       (effects (font (size 1.27 1.27)) hide)
     )
@@
       (effects (font (size 1.27 1.27)) hide)
     )
-    (property "Digikey" "RNCP0603FTD1K00" (at 208.28 123.19 0)
+    (property "Digikey" "RNCP0603FTD1K00CT-ND" (at 208.28 123.19 0)
       (effects (font (size 1.27 1.27)) hide)
     )
@@
       (effects (font (size 1.27 1.27)) hide)
     )
-    (property "Digikey" "RNCP0603FTD1K00" (at 220.98 123.19 0)
-      (effects (font (size 1.27 1.27)) hide)
-    )
+    (property "Digikey" "RNCP0603FTD1K00CT-ND" (at 220.98 123.19 0)
+      (effects (font (size 1.27 1.27)) hide)
+    )
