File: kicad/fan_control.kicad_sch (KiCad schematic)
At the start: 6 parts, among them J209 Conn_01x03, Q202 DMN61D9UWQ-13, Q401 SI7421DN-T1-E3

Commit message: new board
Parts:
- J209: Digikey WM26784TR-ND -> WM26784CT-ND
Changed lines of the file:
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@@
-    (stroke (width 0) (type default))
-  )
-  (wire (pts (xy 142.24 78.74) (xy 142.24 77.47))
     (stroke (width 0) (type default))
   )
@@
   )
   (wire (pts (xy 133.35 96.52) (xy 133.35 97.79))
-    (stroke (width 0) (type default))
-  )
-  (wire (pts (xy 133.35 78.74) (xy 142.24 78.74))
     (stroke (width 0) (type default))
   )
@@
     )
   )
-  (symbol (lib_id "power:PWR_FLAG") (at 142.24 77.47 0) (unit 1)
-    (in_bom yes) (on_board yes) (dnp no) (fields_autoplaced)
-    (property "Reference" "#FLG0201" (at 142.24 75.565 0)
-      (effects (font (size 1.27 1.27)) hide)
-    )
-    (property "Value" "PWR_FLAG" (at 142.24 73.66 0)
-      (effects (font (size 1.27 1.27)))
-    )
-    (property "Footprint" "" (at 142.24 77.47 0)
-      (effects (font (size 1.27 1.27)) hide)
-    )
-    (property "Datasheet" "~" (at 142.24 77.47 0)
-      (effects (font (size 1.27 1.27)) hide)
-    )
-    (pin "1")
-    (instances
-      (project "firewaterburn"
-        (path "/e63e39d7-6ac0-4ffd-8aa3-1841a4541b55/d6846ea7-7fd6-41fd-b190-936bea2a4eb0"
-          (reference "#FLG0201") (unit 1)
-        )
-        (path "/e63e39d7-6ac0-4ffd-8aa3-1841a4541b55/086a34bb-afdd-4e72-a705-1da0ffa64728"
-          (reference "#FLG0701") (unit 1)
-        )
-      )
-    )
-  )
   (symbol (lib_id "power:GND") (at 140.97 115.57 0) (unit 1)
     (in_bom yes) (on_board yes) (dnp no)
@@
       (effects (font (size 1.27 1.27)) hide)
     )
-    (property "Digikey" "WM26784TR-ND" (at 167.64 97.79 0)
+    (property "Digikey" "WM26784CT-ND" (at 167.64 97.79 0)
       (effects (font (size 1.27 1.27)) hide)
     )

Commit message: upgrade 2 KiCAD 8.0
Parts:
- renumbered J209 to J701, Q401 to Q701, Q202 to Q702, R217 to R701, R218 to R702, R219 to R703
