File: kicad/firewaterburn.kicad_sch (KiCad schematic)
At the start: 7 parts, among them P101 USB_C_Plug_USB2.0, U101 TPD4E02B04DQA

Commit message: new board
Parts:
- R101, R102, R103: Digikey 13-RC0402FR-134K7LTR-ND -> 13-RC0402FR-134K7LCT-ND
Other:
- sheet OUTPUT renamed analog
- sheet mcu_n_tft renamed mcu
- sheet analog ports: added none; removed probe6, probe7
- sheet mcu: file mcu_n_tft.kicad_sch -> mcu.kicad_sch
- sheet mcu ports: added WIFI_ENABLE; removed ADC_6, ADC_7, SW_CTRL0
- sheet wifi ports: added WIFI_ENABLE; removed none
Changed lines of the file:
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@@
+    (stroke (width 0) (type default))
+  )
+  (wire (pts (xy 177.8 60.96) (xy 177.8 72.39))
     (stroke (width 0) (type default))
   )
@@
     (stroke (width 0) (type default))
   )
-  (wire (pts (xy 204.47 130.81) (xy 222.25 130.81))
-    (stroke (width 0) (type default))
-  )
   (wire (pts (xy 46.99 140.97) (xy 48.26 140.97))
     (stroke (width 0) (type default))
@@
   )
   (wire (pts (xy 171.45 60.96) (xy 171.45 72.39))
-    (stroke (width 0) (type default))
-  )
-  (wire (pts (xy 204.47 133.35) (xy 222.25 133.35))
     (stroke (width 0) (type default))
   )
@@
       (effects (font (size 1.27 1.27)) hide)
     )
-    (property "Digikey" "13-RC0402FR-134K7LTR-ND" (at 137.16 93.98 0)
+    (property "Digikey" "13-RC0402FR-134K7LCT-ND" (at 137.16 93.98 0)
       (effects (font (size 1.27 1.27)) hide)
     )
@@
       (effects (font (size 1.27 1.27)) hide)
     )
-    (property "Digikey" "13-RC0402FR-134K7LTR-ND" (at 129.54 93.98 0)
+    (property "Digikey" "13-RC0402FR-134K7LCT-ND" (at 129.54 93.98 0)
       (effects (font (size 1.27 1.27)) hide)
     )
@@
       (effects (font (size 1.27 1.27)) hide)
     )
-    (property "Digikey" "13-RC0402FR-134K7LTR-ND" (at 121.92 93.98 0)
+    (property "Digikey" "13-RC0402FR-134K7LCT-ND" (at 121.92 93.98 0)
       (effects (font (size 1.27 1.27)) hide)
     )
@@
     )
   )
-  (sheet (at 151.13 30.48) (size 53.34 30.48)
+  (sheet (at 151.13 40.64) (size 53.34 20.32)
     (stroke (width 0.1524) (type solid))
     (fill (color 7 54 66 1.0000))
-    (property "Sheetname" "wifi" (at 151.13 29.7684 0)
+    (property "Sheetname" "wifi" (at 151.13 39.9284 0)
       (effects (font (size 1.27 1.27)) (justify left bottom))
     )
-    (property "Sheetfile" "wifi.kicad_sch" (at 186.69 27.94 0)
+    (property "Sheetfile" "wifi.kicad_sch" (at 186.69 38.1 0)
       (effects (font (size 1.27 1.27)) (justify left top))
     )
@@
       (effects (font (size 1.27 1.27)) (justify left))
     )
-    (pin "QSPI_DATA3" bidirectional (at 195.58 60.96 270)
-      (effects (font (size 1.27 1.27)) (justify left))
-    )
-    (pin "QSPI_DATA2" bidirectional (at 198.12 60.96 270)
+    (pin "QSPI_DATA3" bidirectional (at 198.12 60.96 270)
+      (effects (font (size 1.27 1.27)) (justify left))
+    )
+    (pin "QSPI_DATA2" bidirectional (at 195.58 60.96 270)
       (effects (font (size 1.27 1.27)) (justify left))
     )
@@
     )
     (pin "COEX_STATUS1" bidirectional (at 168.91 60.96 270)
+      (effects (font (size 1.27 1.27)) (justify left))
+    )
+    (pin "WIFI_ENABLE" input (at 177.8 60.96 270)
       (effects (font (size 1.27 1.27)) (justify left))
     )
@@
     (stroke (width 0) (type solid))
     (fill (color 7 54 66 1.0000))
-    (property "Sheetname" "mcu_n_tft" (at 153.67 82.55 90)
+    (property "Sheetname" "mcu" (at 152.4 72.39 0)
       (effects (font (size 1.27 1.27)) (justify left bottom))
     )
-    (property "Sheetfile" "mcu_n_tft.kicad_sch" (at 151.13 139.0146 0)
+    (property "Sheetfile" "mcu.kicad_sch" (at 151.13 139.0146 0)
       (effects (font (size 1.27 1.27)) (justify left top) hide)
     )
@@
       (effects (font (size 1.27 1.27)) (justify left))
     )
-    (pin "ADC_7" input (at 204.47 133.35 0)
-      (effects (font (size 1.27 1.27)) (justify right))
-    )
-    (pin "ADC_6" input (at 204.47 130.81 0)
-      (effects (font (size 1.27 1.27)) (justify right))
-    )
     (pin "I2C_INT" input (at 151.13 107.95 180)
       (effects (font (size 1.27 1.27)) (justify left))
@@
       (effects (font (size 1.27 1.27)) (justify right))
     )
-    (pin "SW_CTRL0" output (at 201.93 72.39 90)
-      (effects (font (size 1.27 1.27)) (justify right))
-    )
     (pin "TFT_MOSI" input (at 204.47 97.79 0)
       (effects (font (size 1.27 1.27)) (justify right))
@@
     )
     (pin "TFT_~{CS}" input (at 204.47 92.71 0)
+      (effects (font (size 1.27 1.27)) (justify right))
+    )
+    (pin "WIFI_ENABLE" output (at 177.8 72.39 90)
       (effects (font (size 1.27 1.27)) (justify right))
     )
@@
     )
   )
-  (sheet (at 222.25 113.03) (size 17.78 22.86) (fields_autoplaced)
+  (sheet (at 222.25 113.03) (size 17.78 17.78) (fields_autoplaced)
     (stroke (width 0) (type solid))
     (fill (color 7 54 66 1.0000))
-    (property "Sheetname" "OUTPUT" (at 222.25 112.3184 0)
+    (property "Sheetname" "analog" (at 222.25 112.3184 0)
       (effects (font (size 1.27 1.27)) (justify left bottom))
     )
-    (property "Sheetfile" "ntc.kicad_sch" (at 222.25 136.4746 0)
+    (property "Sheetfile" "ntc.kicad_sch" (at 222.25 131.3946 0)
       (effects (font (size 1.27 1.27)) (justify left top) hide)
     )
-    (pin "probe6" output (at 222.25 130.81 180)
-      (effects (font (size 1.27 1.27)) (justify left))
-    )
     (pin "probe3" output (at 222.25 123.19 180)
       (effects (font (size 1.27 1.27)) (justify left))
@@
       (effects (font (size 1.27 1.27)) (justify left))
     )
-    (pin "probe7" output (at 222.25 133.35 180)
-      (effects (font (size 1.27 1.27)) (justify left))
-    )
