File: kicad/lcd.kicad_sch (KiCad schematic)
At the start: 11 parts, among them J501 EA W128064-XALG, U501 MIC2290

Commit message: new board
Parts:
- C4: Digikey 478-7888-2-ND -> 478-7888-1-ND
- C407: Digikey 1276-1067-2-ND -> 1276-1067-1-ND
- C410: Digikey 490-GRM155R61A106ME11DTR-ND -> 490-GRM155R61A106ME11DCT-ND
- C505: Digikey 478-F981C475MMUAJ6TR-ND -> 478-F981C475MMUAJ6CT-ND
- J501: footprint mylib_connector:SFV31R-4STE1HLF -> mylib_connector:F32R-1A7H1-11031
- L501: Digikey 732-4851-2-ND -> 732-4851-1-ND
- R501: Digikey 311-47.5KLRTR-ND -> 311-47.5KLRCT-ND
- R502: Digikey 13-RC0402FR-075KLTR-ND -> 13-RC0402FR-075KLCT-ND
- R503: Digikey 311-910KHRTR-ND -> 311-910KHRCT-ND
- U501: Digikey 576-1076-2-ND -> 576-1076-1-ND
Connections:
- now unconnected: J501.10, J501.14, J501.3, J501.4, J501.5, J501.6, J501.7, J501.8, J501.9
Changed lines of the file:
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@@
       (effects (font (size 1.27 1.27)) hide)
     )
-    (property "Digikey" "490-GRM155R61A106ME11DTR-ND" (at 107.95 48.26 0)
+    (property "Digikey" "490-GRM155R61A106ME11DCT-ND" (at 107.95 48.26 0)
       (effects (font (size 1.27 1.27)) hide)
     )
@@
       (effects (font (size 1.27 1.27)) hide)
     )
-    (property "Digikey" "311-47.5KLRTR-ND" (at 50.8 50.8 0)
+    (property "Digikey" "311-47.5KLRCT-ND" (at 50.8 50.8 0)
       (effects (font (size 1.27 1.27)) hide)
     )
@@
       (effects (font (size 1.27 1.27)) hide)
     )
-    (property "Digikey" "576-1076-2-ND" (at 83.82 50.8 0)
+    (property "Digikey" "576-1076-1-ND" (at 83.82 50.8 0)
       (effects (font (size 1.27 1.27)) hide)
     )
@@
       (effects (font (size 1.27 1.27)) hide)
     )
-    (property "Digikey" "13-RC0402FR-075KLTR-ND" (at 50.8 60.96 0)
+    (property "Digikey" "13-RC0402FR-075KLCT-ND" (at 50.8 60.96 0)
       (effects (font (size 1.27 1.27)) hide)
     )
@@
       (effects (font (size 1.27 1.27)) hide)
     )
-    (property "Digikey" "478-F981C475MMUAJ6TR-ND" (at 191.77 125.73 0)
+    (property "Digikey" "478-F981C475MMUAJ6CT-ND" (at 191.77 125.73 0)
       (effects (font (size 1.27 1.27)) hide)
     )
@@
       (effects (font (size 1.27 1.27)) hide)
     )
-    (property "Digikey" "311-910KHRTR-ND" (at 223.52 124.46 0)
+    (property "Digikey" "311-910KHRCT-ND" (at 223.52 124.46 0)
       (effects (font (size 1.27 1.27)) hide)
     )
@@
       (effects (font (size 1.27 1.27)) hide)
     )
-    (property "Digikey" "478-7888-2-ND" (at 120.65 48.26 0)
+    (property "Digikey" "478-7888-1-ND" (at 120.65 48.26 0)
       (effects (font (size 1.27 1.27)) hide)
     )
@@
       (effects (font (size 1.27 1.27)) hide)
     )
-    (property "Digikey" "732-4851-2-ND" (at 67.31 53.34 90)
+    (property "Digikey" "732-4851-1-ND" (at 67.31 53.34 90)
       (effects (font (size 1.27 1.27)) hide)
     )
@@
       (effects (font (size 1.27 1.27)) (justify left))
     )
-    (property "Footprint" "mylib_connector:SFV31R-4STE1HLF" (at 191.135 90.805 0)
+    (property "Footprint" "mylib_connector:F32R-1A7H1-11031" (at 191.135 90.805 0)
       (effects (font (size 1.27 1.27)) hide)
     )
@@
       (effects (font (size 1.27 1.27)) hide)
     )
-    (property "Digikey" "1276-1067-2-ND" (at 35.56 46.99 0)
-      (effects (font (size 1.27 1.27)) hide)
-    )
+    (property "Digikey" "1276-1067-1-ND" (at 35.56 46.99 0)
+      (effects (font (size 1.27 1.27)) hide)
+    )

Commit message: upgrade 2 KiCAD 8.0
Parts:
- renumbered C407 to C501, C410 to C502, C4 to C503, C4 to C504
