File: kicad/mcu.kicad_sch (KiCad schematic)
At the start: 18 parts, among them J301 Conn_ARM_SWD_TagConnect_TC2030, J303 Conn_02x10_Odd_Even, SW301 SW_Push, U301 BL654, Y301 Crystal

Commit message: upgrade 2 KiCAD 8.0
Parts:
- added U1: ~, mylib_ic:BL5340, symbol mylib_ic:BL5340
- renumbered C5 to C301, C4 to C302, C4 to C306, D401 to D301, D402 to D302, R101 to R301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
Connections:
- net GND: now also U1.1 (GND), U1.19 (GND), U1.21 (GND), U1.29 (GND), U1.30 (GND), U1.33 (GND), U1.39 (GND), U1.44 (GND), U1.59 (GND), U1.66 (GND), U1.67 (GND), U1.68 (GND)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
