File: kicad/ntc.kicad_sch (KiCad schematic)
At the start: 24 parts, among them J201 AudioJack2_SwitchT, J202 AudioJack2_SwitchT, J203 AudioJack2_SwitchT, J204 AudioJack2_SwitchT, J205 AudioJack2_SwitchT, J206 AudioJack2_SwitchT, J207 AudioJack2_SwitchT, J208 AudioJack2_SwitchT

Commit message: new board
Parts:
- removed J207, J208: AudioJack2_SwitchT, mylib_connector:MJ-2523, symbol Connector_Audio:AudioJack2_SwitchT
- removed R211, R212: 4k42, Resistor_SMD:R_0603_1608Metric, symbol Device:R
- removed R215, R216: 3k4, Resistor_SMD:R_0603_1608Metric, symbol Device:R
