File: kicad/pwr_supply.kicad_sch (KiCad schematic)
At the start: 31 parts, among them Q401 SI7421DN-T1-E3, U401 LT3973-3.3, U402 STUSB4500QTR, U403 LM2775DSG

Commit message: new board
Parts:
- removed TP402, TP403, TP404, TP405: TestPoint, TestPoint:TestPoint_Keystone_5015_Micro-Minature, symbol Connector:TestPoint
- C403, C409: Digikey CL10A105KA8NNNC -> 1276-1102-1-ND
- C406, C407: Digikey 1276-1067-2-ND -> 1276-1067-1-ND
- R407: Digikey 1292-WR04X1003FTLTR-ND -> 1292-WR04X1003FTLCT-ND
- R408, R409: Digikey RNCP0603FTD1K00 -> RNCP0603FTD1K00CT-ND
Changed lines of the file:
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@@
-    (stroke (width 0) (type default))
-  )
-  (wire (pts (xy 240.03 55.88) (xy 240.03 46.99))
     (stroke (width 0) (type default))
   )
@@
     (stroke (width 0) (type default))
   )
-  (wire (pts (xy 119.38 43.18) (xy 123.19 43.18))
-    (stroke (width 0) (type default))
-  )
   (wire (pts (xy 189.23 123.19) (xy 189.23 120.65))
     (stroke (width 0) (type default))
@@
     (stroke (width 0) (type default))
   )
-  (wire (pts (xy 31.75 43.18) (xy 45.72 43.18))
-    (stroke (width 0) (type default))
-  )
   (wire (pts (xy 69.85 109.22) (xy 69.85 114.3))
     (stroke (width 0) (type default))
@@
     (stroke (width 0) (type default))
   )
-  (wire (pts (xy 228.6 118.11) (xy 233.68 118.11))
-    (stroke (width 0) (type default))
-  )
   (wire (pts (xy 73.66 69.85) (xy 73.66 73.66))
     (stroke (width 0) (type default))
@@
     (stroke (width 0) (type default))
   )
-  (wire (pts (xy 233.68 118.11) (xy 233.68 115.57))
-    (stroke (width 0) (type default))
-  )
   (wire (pts (xy 78.74 43.18) (xy 78.74 49.53))
     (stroke (width 0) (type default))
@@
     (stroke (width 0) (type default))
   )
-  (wire (pts (xy 234.95 55.88) (xy 240.03 55.88))
-    (stroke (width 0) (type default))
-  )
   (wire (pts (xy 77.47 160.02) (xy 77.47 163.83))
-    (stroke (width 0) (type default))
-  )
-  (wire (pts (xy 31.75 43.18) (xy 31.75 40.64))
-    (stroke (width 0) (type default))
-  )
-  (wire (pts (xy 123.19 43.18) (xy 123.19 40.64))
     (stroke (width 0) (type default))
   )
@@
       (effects (font (size 1.27 1.27)) hide)
     )
-    (property "Digikey" "1276-1067-2-ND" (at 55.88 97.79 0)
+    (property "Digikey" "1276-1067-1-ND" (at 55.88 97.79 0)
       (effects (font (size 1.27 1.27)) hide)
     )
@@
       (effects (font (size 1.27 1.27)) hide)
     )
-    (property "Digikey" "RNCP0603FTD1K00" (at 90.17 156.21 0)
+    (property "Digikey" "RNCP0603FTD1K00CT-ND" (at 90.17 156.21 0)
       (effects (font (size 1.27 1.27)) hide)
     )
@@
       (effects (font (size 1.27 1.27)) hide)
     )
-    (property "Digikey" "CL10A105KA8NNNC" (at 218.44 125.73 0)
+    (property "Digikey" "1276-1102-1-ND" (at 218.44 125.73 0)
       (effects (font (size 1.27 1.27)) hide)
     )
@@
       (effects (font (size 1.27 1.27)) hide)
     )
-    (property "Digikey" "1292-WR04X1003FTLTR-ND" (at 119.38 115.57 0)
+    (property "Digikey" "1292-WR04X1003FTLCT-ND" (at 119.38 115.57 0)
       (effects (font (size 1.27 1.27)) hide)
     )
@@
       (effects (font (size 1.27 1.27)) hide)
     )
-    (property "Digikey" "CL10A105KA8NNNC" (at 45.72 60.96 0)
+    (property "Digikey" "1276-1102-1-ND" (at 45.72 60.96 0)
       (effects (font (size 1.27 1.27)) hide)
     )
@@
         (path "/e63e39d7-6ac0-4ffd-8aa3-1841a4541b55/da8e08cc-b8fa-44d2-9f6f-15fecbf9ecc5"
           (reference "#PWR0412") (unit 1)
-        )
-      )
-    )
-  )
-  (symbol (lib_id "Connector:TestPoint") (at 31.75 40.64 0) (unit 1)
-    (in_bom yes) (on_board yes) (dnp no) (fields_autoplaced)
-    (property "Reference" "TP402" (at 34.29 36.703 0)
-      (effects (font (size 1.27 1.27)) (justify left))
-    )
-    (property "Value" "TestPoint" (at 34.29 39.243 0)
-      (effects (font (size 1.27 1.27)) (justify left))
-    )
-    (property "Footprint" "TestPoint:TestPoint_Keystone_5015_Micro-Minature" (at 36.83 40.64 0)
-      (effects (font (size 1.27 1.27)) hide)
-    )
-    (property "Datasheet" "~" (at 36.83 40.64 0)
-      (effects (font (size 1.27 1.27)) hide)
-    )
-    (property "Digikey" "36-5015CT-ND" (at 31.75 40.64 0)
-      (effects (font (size 1.27 1.27)) hide)
-    )
-    (pin "1")
-    (instances
-      (project "firewaterburn"
-        (path "/e63e39d7-6ac0-4ffd-8aa3-1841a4541b55/da8e08cc-b8fa-44d2-9f6f-15fecbf9ecc5"
-          (reference "TP402") (unit 1)
         )
       )
@@
     )
   )
-  (symbol (lib_id "Connector:TestPoint") (at 240.03 46.99 0) (unit 1)
-    (in_bom yes) (on_board yes) (dnp no) (fields_autoplaced)
-    (property "Reference" "TP404" (at 242.57 43.053 0)
-      (effects (font (size 1.27 1.27)) (justify left))
-    )
-    (property "Value" "TestPoint" (at 242.57 45.593 0)
-      (effects (font (size 1.27 1.27)) (justify left))
-    )
-    (property "Footprint" "TestPoint:TestPoint_Keystone_5015_Micro-Minature" (at 245.11 46.99 0)
-      (effects (font (size 1.27 1.27)) hide)
-    )
-    (property "Datasheet" "~" (at 245.11 46.99 0)
-      (effects (font (size 1.27 1.27)) hide)
-    )
-    (property "Digikey" "36-5015CT-ND" (at 240.03 46.99 0)
-      (effects (font (size 1.27 1.27)) hide)
-    )
-    (pin "1")
-    (instances
-      (project "firewaterburn"
-        (path "/e63e39d7-6ac0-4ffd-8aa3-1841a4541b55/da8e08cc-b8fa-44d2-9f6f-15fecbf9ecc5"
-          (reference "TP404") (unit 1)
-        )
-      )
-    )
-  )
   (symbol (lib_id "power:+5V") (at 228.6 115.57 0) (unit 1)
     (in_bom yes) (on_board yes) (dnp no)
@@
       (effects (font (size 1.27 1.27)) hide)
     )
-    (property "Digikey" "1276-1067-2-ND" (at 45.72 97.79 0)
+    (property "Digikey" "1276-1067-1-ND" (at 45.72 97.79 0)
       (effects (font (size 1.27 1.27)) hide)
     )
@@
       (effects (font (size 1.27 1.27)) hide)
     )
-    (property "Digikey" "RNCP0603FTD1K00" (at 77.47 156.21 0)
+    (property "Digikey" "RNCP0603FTD1K00CT-ND" (at 77.47 156.21 0)
       (effects (font (size 1.27 1.27)) hide)
     )
@@
         (path "/e63e39d7-6ac0-4ffd-8aa3-1841a4541b55/da8e08cc-b8fa-44d2-9f6f-15fecbf9ecc5"
           (reference "R408") (unit 1)
-        )
-      )
-    )
-  )
-  (symbol (lib_id "Connector:TestPoint") (at 233.68 115.57 0) (unit 1)
-    (in_bom yes) (on_board yes) (dnp no) (fields_autoplaced)
-    (property "Reference" "TP405" (at 236.22 111.633 0)
-      (effects (font (size 1.27 1.27)) (justify left))
-    )
-    (property "Value" "TestPoint" (at 236.22 114.173 0)
-      (effects (font (size 1.27 1.27)) (justify left))
-    )
-    (property "Footprint" "TestPoint:TestPoint_Keystone_5015_Micro-Minature" (at 238.76 115.57 0)
-      (effects (font (size 1.27 1.27)) hide)
-    )
-    (property "Datasheet" "~" (at 238.76 115.57 0)
-      (effects (font (size 1.27 1.27)) hide)
-    )
-    (property "Digikey" "36-5015CT-ND" (at 233.68 115.57 0)
-      (effects (font (size 1.27 1.27)) hide)
-    )
-    (pin "1")
-    (instances
-      (project "firewaterburn"
-        (path "/e63e39d7-6ac0-4ffd-8aa3-1841a4541b55/da8e08cc-b8fa-44d2-9f6f-15fecbf9ecc5"
-          (reference "TP405") (unit 1)
         )
       )
@@
         )
       )
-    )
-  )
-  (symbol (lib_id "Connector:TestPoint") (at 123.19 40.64 0) (unit 1)
-    (in_bom yes) (on_board yes) (dnp no) (fields_autoplaced)
-    (property "Reference" "TP403" (at 125.73 36.703 0)
-      (effects (font (size 1.27 1.27)) (justify left))
-    )
-    (property "Value" "TestPoint" (at 125.73 39.243 0)
-      (effects (font (size 1.27 1.27)) (justify left))
-    )
-    (property "Footprint" "TestPoint:TestPoint_Keystone_5015_Micro-Minature" (at 128.27 40.64 0)
-      (effects (font (size 1.27 1.27)) hide)
-    )
-    (property "Datasheet" "~" (at 128.27 40.64 0)
-      (effects (font (size 1.27 1.27)) hide)
-    )
-    (property "Digikey" "36-5015CT-ND" (at 123.19 40.64 0)
-      (effects (font (size 1.27 1.27)) hide)
-    )
-    (pin "1")
-    (instances
-      (project "firewaterburn"
-        (path "/e63e39d7-6ac0-4ffd-8aa3-1841a4541b55/da8e08cc-b8fa-44d2-9f6f-15fecbf9ecc5"
-          (reference "TP403") (unit 1)
-        )
-      )

Commit message: upgrade 2 KiCAD 8.0
Parts:
- renumbered C303 to C404
